Commit message: 小车+蛇臂，成功

File: src/raphael_robot_description/urdf/10_snake/11_snake_joints.xacro (robot description, xacro)
@@ -110,5 +110,5 @@
             <limit effort="${effort}" velocity="${velocity}" lower="${-rad_135}" upper="${rad_135}"/>
         </joint>
-        <!-- link10 -> link11 (分叉1) -->
+        <!-- link10 -> link11 【主动驱动关节，电机驱动】 -->
         <joint name="${prefix}_link10_link11_joint" type="revolute">
             <parent link="${prefix}_link10"/>
@@ -116,7 +116,7 @@
             <origin xyz="${x_offset_10_11} 0 0" rpy="0 0 0"/>
             <axis xyz="0 1 0"/>
-            <limit effort="${effort}" velocity="${velocity}" lower="0" upper="${-rad_fork}"/>
+            <limit effort="${effort}" velocity="${velocity}" lower="${-rad_fork}" upper="0"/>
         </joint>
-        <!-- link10 -> link12 (分叉2) -->
+        <!-- link10 -> link12 【mimic镜像跟随，剪刀另一侧刀片】 -->
         <joint name="${prefix}_link10_link12_joint" type="revolute">
             <parent link="${prefix}_link10"/>
@@ -124,5 +124,6 @@
             <origin xyz="${x_offset_10_12} 0 0" rpy="0 0 0"/>
             <axis xyz="0 1 0"/>
-            <limit effort="${effort}" velocity="${velocity}" lower="${rad_fork}" upper="0"/>
+            <limit effort="${effort}" velocity="${velocity}" lower="0" upper="${rad_fork}"/>
+            <mimic joint="${prefix}_link10_link11_joint" multiplier="-1.0" offset="0.0"/>
         </joint>
     </xacro:macro>

File: src/raphael_robot_description/urdf/10_snake/89_snake_robot.ros2_control.xacro (robot description, xacro)
@@ -1,5 +1,63 @@
 <?xml version="1.0"?>
 <robot xmlns:xacro="http://www.ros.org/wiki/xacro">
-    <ros2_control name="SnakeCtrl" type="system">
+    <ros2_control name="SnakeHardwareInterface" type="system">
+        <hardware>
+            <plugin>mock_components/GenericSystem</plugin>
+            <param name="calculate_dynamics">true</param>
+        </hardware>
+        <joint name="s1_link01_link02_joint">
+            <command_interface name="velocity"/>
+            <state_interface name="velocity"/>
+            <state_interface name="position"/>
+        </joint>
+        <joint name="s1_link02_link03_joint">
+            <command_interface name="velocity"/>
+            <state_interface name="velocity"/>
+            <state_interface name="position"/>
+        </joint>
+        <joint name="s1_link03_link04_joint">
+            <command_interface name="velocity"/>
+            <state_interface name="velocity"/>
+            <state_interface name="position"/>
+        </joint>
+        <joint name="s1_link04_link05_joint">
+            <command_interface name="velocity"/>
+            <state_interface name="velocity"/>
+            <state_interface name="position"/>
+        </joint>
+        <joint name="s1_link05_link06_joint">
+            <command_interface name="velocity"/>
+            <state_interface name="velocity"/>
+            <state_interface name="position"/>
+        </joint>
+        <joint name="s1_link06_link07_joint">
+            <command_interface name="velocity"/>
+            <state_interface name="velocity"/>
+            <state_interface name="position"/>
+        </joint>
+        <joint name="s1_link07_link08_joint">
+            <command_interface name="velocity"/>
+            <state_interface name="velocity"/>
+            <state_interface name="position"/>
+        </joint>
+        <joint name="s1_link08_link09_joint">
+            <command_interface name="velocity"/>
+            <state_interface name="velocity"/>
+            <state_interface name="position"/>
+        </joint>
+        <joint name="s1_link09b_link10_joint">
+            <command_interface name="velocity"/>
+            <state_interface name="velocity"/>
+            <state_interface name="position"/>
+        </joint>
+        <joint name="s1_link10_link11_joint">
+            <command_interface name="velocity"/>
+            <state_interface name="velocity"/>
+            <state_interface name="position"/>
+        </joint>
+        <joint name="s1_link10_link12_joint">
+            <state_interface name="velocity"/>
+            <state_interface name="position"/>
+        </joint>
     </ros2_control>
 </robot>

File: src/raphael_robot_description/urdf/raphael_robot.urdf.xacro (robot description, xacro)
@@ -2,11 +2,18 @@
 <robot name="raphael_robot" xmlns:xacro="http://www.ros.org/wiki/xacro">
     <!-- 导入snake_robot -->
-    <xacro:include filename="$(find raphael_robot_description)/urdf/01_snake/99_snake_robot.urdf.xacro"/>
+    <xacro:include filename="$(find raphael_robot_description)/urdf/10_snake/99_snake_robot.urdf.xacro"/>
+    <!-- 导入tricycle -->
+    <xacro:include filename="$(find raphael_robot_description)/urdf/40_tricycle/99_tricycle_robot.urdf.xacro"/>
     <!-- raphael_robot 总装基点-->
     <link name="base_footprint"/>
-    <joint name="base_snake_joints" type="fixed">
+    <joint name="base_tricycle_joints" type="fixed">
         <parent link="base_footprint"/>
-        <child link="base_footprint_snake"/>
+        <child link="base_footprint_tricycle"/>
         <origin xyz="0 0 0" rpy="0 0 0"/>
     </joint>
+    <joint name="base_tricycle_snake_joints" type="fixed">
+        <parent link="base_footprint_tricycle"/>
+        <child link="base_footprint_snake"/>
+        <origin xyz="0 0 0.033" rpy="0 0 0"/>
+    </joint>
 </robot>
