Commit message: 提交

File: src/raphael_robot_description/urdf/10_snake/69_snake_robot.xacro (robot description, xacro)
@@ -18,8 +18,10 @@
     <!-- 17 生成 base_footprint_snake 固定基座 -->
     <link name="base_footprint_snake"/>
-    <joint name="base_s1_link00" type="fixed">
+    <joint name="base_s1_link00" type="prismatic">
         <parent link="base_footprint_snake"/>
         <child link="s1_link00"/>
         <origin xyz="0 0 0" rpy="0 0 0"/>
+        <axis xyz="1 0 0"/>
+        <limit lower="-0.1" upper="0.1" effort="1000" velocity="10"/>
     </joint>
 </robot>

File: src/raphael_robot_description/urdf/10_snake/89_snake_robot.ros2_control.xacro (robot description, xacro)
@@ -1,61 +1,85 @@
 <?xml version="1.0"?>
 <robot xmlns:xacro="http://www.ros.org/wiki/xacro">
-    <ros2_control name="SnakeHardwareInterface" type="system">
+    <!--    <ros2_control name="SnakeHardware" type="system">-->
+    <!--        <hardware>-->
+    <!--            <plugin>snake_hardware/SnakeHardwareInterface</plugin>-->
+    <!--            <param name="st3215_port">/dev/ttyACM0</param>-->
+    <!--            <param name="baud">1000000</param>-->
+    <!--            <param name="s1_motor_06_07">6</param>-->
+    <!--            <param name="s1_motor_07_08">7</param>-->
+    <!--            <param name="s1_motor_08_09">8</param>-->
+    <!--            <param name="s1_motor_09b_10">9</param>-->
+    <!--            <param name="s1_motor_10_11">10</param>-->
+    <!--        </hardware>-->
+    <!--        <joint name="s1_link06_link07_joint">-->
+    <!--            <command_interface name="position"/>-->
+    <!--            <state_interface name="position"/>-->
+    <!--        </joint>-->
+    <!--        <joint name="s1_link07_link08_joint">-->
+    <!--            <command_interface name="position"/>-->
+    <!--            <state_interface name="position"/>-->
+    <!--        </joint>-->
+    <!--        <joint name="s1_link08_link09_joint">-->
+    <!--            <command_interface name="position"/>-->
+    <!--            <state_interface name="position"/>-->
+    <!--        </joint>-->
+    <!--        <joint name="s1_link09b_link10_joint">-->
+    <!--            <command_interface name="position"/>-->
+    <!--            <state_interface name="position"/>-->
+    <!--        </joint>-->
+    <!--        <joint name="s1_link10_link11_joint">-->
+    <!--            <command_interface name="position"/>-->
+    <!--            <state_interface name="position"/>-->
+    <!--        </joint>-->
+    <!--    </ros2_control>-->
+    <!--    仿真/Mock 硬件接口配置-->
+    <ros2_control name="SnakeHardwareMock" type="system">
         <hardware>
             <plugin>mock_components/GenericSystem</plugin>
             <param name="calculate_dynamics">true</param>
         </hardware>
+        <joint name="base_s1_link00">
+            <command_interface name="position"/>
+            <state_interface name="position"/>
+        </joint>
         <joint name="s1_link01_link02_joint">
-            <command_interface name="velocity"/>
-            <state_interface name="velocity"/>
+            <command_interface name="position"/>
             <state_interface name="position"/>
         </joint>
         <joint name="s1_link02_link03_joint">
-            <command_interface name="velocity"/>
-            <state_interface name="velocity"/>
+            <command_interface name="position"/>
             <state_interface name="position"/>
         </joint>
         <joint name="s1_link03_link04_joint">
-            <command_interface name="velocity"/>
-            <state_interface name="velocity"/>
+            <command_interface name="position"/>
             <state_interface name="position"/>
         </joint>
         <joint name="s1_link04_link05_joint">
-            <command_interface name="velocity"/>
-            <state_interface name="velocity"/>
+            <command_interface name="position"/>
             <state_interface name="position"/>
         </joint>
         <joint name="s1_link05_link06_joint">
-            <command_interface name="velocity"/>
-            <state_interface name="velocity"/>
+            <command_interface name="position"/>
             <state_interface name="position"/>
         </joint>
-        <joint name="s1_link06_link07_joint">
-            <command_interface name="velocity"/>
-            <state_interface name="velocity"/>
+        <!--  ========================== 以下就有足够的电机可以匹配了 ========================-->
+        <joint name="s1_link06_link07_joint">-->
+            <command_interface name="position"/>
             <state_interface name="position"/>
         </joint>
         <joint name="s1_link07_link08_joint">
-            <command_interface name="velocity"/>
-            <state_interface name="velocity"/>
+            <command_interface name="position"/>
             <state_interface name="position"/>
         </joint>
         <joint name="s1_link08_link09_joint">
-            <command_interface name="velocity"/>
-            <state_interface name="velocity"/>
+            <command_interface name="position"/>
             <state_interface name="position"/>
         </joint>
         <joint name="s1_link09b_link10_joint">
-            <command_interface name="velocity"/>
-            <state_interface name="velocity"/>
+            <command_interface name="position"/>
             <state_interface name="position"/>
         </joint>
         <joint name="s1_link10_link11_joint">
-            <command_interface name="velocity"/>
-            <state_interface name="velocity"/>
-            <state_interface name="position"/>
-        </joint>
-        <joint name="s1_link10_link12_joint">
-            <state_interface name="velocity"/>
+            <command_interface name="position"/>
             <state_interface name="position"/>
         </joint>

File: src/raphael_robot_description/urdf/40_tricycle/89_mobile_base.ros2_control.xacro (robot description, xacro)
@@ -1,9 +1,15 @@
 <?xml version="1.0"?>
 <robot xmlns:xacro="http://www.ros.org/wiki/xacro">
-    <ros2_control name="TricycleHardwareInterface" type="system">
+    <ros2_control name="TricycleHardware" type="system">
         <hardware>
             <plugin>mock_components/GenericSystem</plugin>
             <param name="calculate_dynamics">true</param>
         </hardware>
+        <!--        <hardware>-->
+        <!--            <plugin>tricycle_hardware/TricycleHardwareInterface</plugin>-->
+        <!--            <param name="left_motor_id">10</param>-->
+        <!--            <param name="right_motor_id">20</param>-->
+        <!--            <param name="st3215_port">/dev/ttyUSB2</param>-->
+        <!--        </hardware>-->
         <joint name="base_right_wheel_joint">
             <command_interface name="velocity"/>
