Commit message: gazebo_ros2_control， 没完成，先保存在这里

File: src/raphael_robot_description/urdf/10_snake/00_snake_params.xacro (robot description, xacro)
@@ -3,47 +3,47 @@
 <robot xmlns:xacro="http://www.ros.org/wiki/xacro">
     <!-- ====================== 各连杆质量 m(kg) ====================== -->
-    <xacro:property name="link0_m" value="0.10"/>
-    <xacro:property name="link1_m" value="0.10"/>
-    <xacro:property name="link2_m" value="0.10"/>
-    <xacro:property name="link3_m" value="0.10"/>
-    <xacro:property name="link4_m" value="0.10"/>
-    <xacro:property name="link5_m" value="0.10"/>
-    <xacro:property name="link6_m" value="0.10"/>
-    <xacro:property name="link7_m" value="0.10"/>
-    <xacro:property name="link8_m" value="0.10"/>
-    <xacro:property name="link9_m" value="0.10"/>
-    <xacro:property name="link10_m" value="0.10"/>
-    <xacro:property name="link11_m" value="0.10"/>
-    <xacro:property name="link12_m" value="0.10"/>
-    <xacro:property name="link13_m" value="0.10"/>
+    <xacro:property name="link00_m" value="0.0258"/>
+    <xacro:property name="link01_m" value="0.00170"/>
+    <xacro:property name="link02_m" value="0.00170"/>
+    <xacro:property name="link03_m" value="0.0123"/>
+    <xacro:property name="link04_m" value="0.00170"/>
+    <xacro:property name="link05_m" value="0.00635"/>
+    <xacro:property name="link06_m" value="0.00170"/>
+    <xacro:property name="link07_m" value="0.00170"/>
+    <xacro:property name="link08_m" value="0.00170"/>
+    <xacro:property name="link09_m" value="0.00686"/>
+    <xacro:property name="link09b_m" value="0.000671"/>
+    <xacro:property name="link10_m" value="0.00619"/>
+    <xacro:property name="link11_m" value="0.00671"/>
+    <xacro:property name="link12_m" value="0.00671"/>
     <!-- ====================== 各连杆外半径 r(m) ====================== -->
-    <xacro:property name="link0_r" value="0.0078"/>
-    <xacro:property name="link1_r" value="0.0078"/>
-    <xacro:property name="link2_r" value="0.0078"/>
-    <xacro:property name="link3_r" value="0.0078"/>
-    <xacro:property name="link4_r" value="0.0078"/>
-    <xacro:property name="link5_r" value="0.0078"/>
-    <xacro:property name="link6_r" value="0.0078"/>
-    <xacro:property name="link7_r" value="0.0078"/>
-    <xacro:property name="link8_r" value="0.0078"/>
-    <xacro:property name="link9_r" value="0.0078"/>
-    <xacro:property name="link10_r" value="0.0078"/>
-    <xacro:property name="link11_r" value="0.0078"/>
-    <xacro:property name="link12_r" value="0.0078"/>
-    <xacro:property name="link13_r" value="0.0078"/>
+    <xacro:property name="link00_r" value="0.004"/>
+    <xacro:property name="link01_r" value="0.004"/>
+    <xacro:property name="link02_r" value="0.004"/>
+    <xacro:property name="link03_r" value="0.004"/>
+    <xacro:property name="link04_r" value="0.004"/>
+    <xacro:property name="link05_r" value="0.004"/>
+    <xacro:property name="link06_r" value="0.004"/>
+    <xacro:property name="link07_r" value="0.004"/>
+    <xacro:property name="link08_r" value="0.004"/>
+    <xacro:property name="link09_r" value="0.004"/>
+    <xacro:property name="link09b_r" value="0.004"/>
+    <xacro:property name="link10_r" value="0.004"/>
+    <xacro:property name="link11_r" value="0.004"/>
+    <xacro:property name="link12_r" value="0.004"/>
     <!-- ====================== 各连杆总长 l(m) ====================== -->
-    <xacro:property name="link0_l" value="0.285"/>
-    <xacro:property name="link1_l" value="0.1200"/>
-    <xacro:property name="link2_l" value="0.1180"/>
-    <xacro:property name="link3_l" value="0.1160"/>
-    <xacro:property name="link4_l" value="0.1150"/>
-    <xacro:property name="link5_l" value="0.1140"/>
-    <xacro:property name="link6_l" value="0.1130"/>
-    <xacro:property name="link7_l" value="0.1120"/>
-    <xacro:property name="link8_l" value="0.1110"/>
-    <xacro:property name="link9_l" value="0.1100"/>
-    <xacro:property name="link10_l" value="0.1090"/>
-    <xacro:property name="link11_l" value="0.1080"/>
-    <xacro:property name="link12_l" value="0.1070"/>
-    <xacro:property name="link13_l" value="0.1000"/>
+    <xacro:property name="link00_l" value="0.05"/>
+    <xacro:property name="link01_l" value="0.0033"/>
+    <xacro:property name="link02_l" value="0.0033"/>
+    <xacro:property name="link03_l" value="0.0238"/>
+    <xacro:property name="link04_l" value="0.0033"/>
+    <xacro:property name="link05_l" value="0.0123"/>
+    <xacro:property name="link06_l" value="0.0033"/>
+    <xacro:property name="link07_l" value="0.0033"/>
+    <xacro:property name="link08_l" value="0.0033"/>
+    <xacro:property name="link09_l" value="0.0133"/>
+    <xacro:property name="link09b_l" value="0.0013"/>
+    <xacro:property name="link10_l" value="0.012"/>
+    <xacro:property name="link11_l" value="0.013"/>
+    <xacro:property name="link12_l" value="0.013"/>
 </robot>

File: src/raphael_robot_description/urdf/10_snake/10_snake_links.xacro (robot description, xacro)
@@ -16,4 +16,5 @@
                 <origin xyz="0 0 0" rpy="0 ${pi} 0"/>
             </collision>
+            <xacro:snake_cylinder_inertia m="${link00_m}" r="${link00_r}" l="${link00_l}" o_xyz="0 0 0" o_rpy="0 ${pi} 0"/>
         </link>
         <link name="${prefix}_link01">
@@ -31,4 +32,5 @@
                 <origin xyz="0 0 0" rpy="0 0 0"/>
             </collision>
+            <xacro:snake_cylinder_inertia m="${link01_m}" r="${link01_r}" l="${link01_l}" o_xyz="0 0 0" o_rpy="0 0 0"/>
         </link>
         <link name="${prefix}_link02">
@@ -46,4 +48,5 @@
                 <origin xyz="0 0 0" rpy="0 0 0"/>
             </collision>
+            <xacro:snake_cylinder_inertia m="${link02_m}" r="${link02_r}" l="${link02_l}" o_xyz="0 0 0" o_rpy="0 0 0"/>
         </link>
         <link name="${prefix}_link03">
@@ -61,4 +64,5 @@
                 <origin xyz="0 0 0" rpy="0 0 0"/>
             </collision>
+            <xacro:snake_cylinder_inertia m="${link03_m}" r="${link03_r}" l="${link03_l}" o_xyz="0 0 0" o_rpy="0 0 0"/>
         </link>
         <link name="${prefix}_link04">
@@ -76,4 +80,5 @@
                 <origin xyz="0 0 0" rpy="0 0 0"/>
             </collision>
+            <xacro:snake_cylinder_inertia m="${link04_m}" r="${link04_r}" l="${link04_l}" o_xyz="0 0 0" o_rpy="0 0 0"/>
         </link>
         <link name="${prefix}_link05">
@@ -91,4 +96,5 @@
                 <origin xyz="0 0 0" rpy="0 0 0"/>
             </collision>
+            <xacro:snake_cylinder_inertia m="${link05_m}" r="${link05_r}" l="${link05_l}" o_xyz="0 0 0" o_rpy="0 0 0"/>
         </link>
         <link name="${prefix}_link06">
@@ -106,4 +112,5 @@
                 <origin xyz="0 0 0" rpy="0 0 0"/>
             </collision>
+            <xacro:snake_cylinder_inertia m="${link06_m}" r="${link06_r}" l="${link06_l}" o_xyz="0 0 0" o_rpy="0 0 0"/>
         </link>
         <link name="${prefix}_link07">
@@ -121,4 +128,5 @@
                 <origin xyz="0 0 0" rpy="0 0 0"/>
             </collision>
+            <xacro:snake_cylinder_inertia m="${link07_m}" r="${link07_r}" l="${link07_l}" o_xyz="0 0 0" o_rpy="0 0 0"/>
         </link>
         <link name="${prefix}_link08">
@@ -136,4 +144,5 @@
                 <origin xyz="0 0 0" rpy="0 0 0"/>
             </collision>
+            <xacro:snake_cylinder_inertia m="${link08_m}" r="${link08_r}" l="${link08_l}" o_xyz="0 0 0" o_rpy="0 0 0"/>
         </link>
         <link name="${prefix}_link09">
@@ -151,4 +160,5 @@
                 <origin xyz="0 0 0" rpy="0 0 0"/>
             </collision>
+            <xacro:snake_cylinder_inertia m="${link09_m}" r="${link09_r}" l="${link09_l}" o_xyz="0 0 0" o_rpy="0 0 0"/>
         </link>
         <link name="${prefix}_link09b">
@@ -166,4 +176,5 @@
                 <origin xyz="0 0 0" rpy="0 0 0"/>
             </collision>
+            <xacro:snake_cylinder_inertia m="${link09b_m}" r="${link09b_r}" l="${link09b_l}" o_xyz="0 0 0" o_rpy="0 0 0"/>
         </link>
         <link name="${prefix}_link10">
@@ -181,4 +192,5 @@
                 <origin xyz="0 0 0" rpy="0 0 0"/>
             </collision>
+            <xacro:snake_cylinder_inertia m="${link10_m}" r="${link10_r}" l="${link10_l}" o_xyz="0 0 0" o_rpy="0 0 0"/>
         </link>
         <link name="${prefix}_link11">
@@ -196,4 +208,5 @@
                 <origin xyz="0 0 0" rpy="0 0 0"/>
             </collision>
+            <xacro:snake_cylinder_inertia m="${link11_m}" r="${link11_r}" l="${link11_l}" o_xyz="0 0 0" o_rpy="0 0 0"/>
         </link>
         <link name="${prefix}_link12">
@@ -211,4 +224,5 @@
                 <origin xyz="0 0 0" rpy="0 0 0"/>
             </collision>
+            <xacro:snake_cylinder_inertia m="${link12_m}" r="${link12_r}" l="${link12_l}" o_xyz="0 0 0" o_rpy="0 0 0"/>
         </link>
     </xacro:macro>

File: src/raphael_robot_description/urdf/10_snake/11_snake_joints.xacro (robot description, xacro)
@@ -19,5 +19,5 @@
     <xacro:property name="effort" value="1000"/>
     <!-- ========= 最大速度 rad/s ======== -->
-    <xacro:property name="velocity" value="0.5"/>
+    <xacro:property name="velocity" value="6"/>
     <!-- ========= 旋转角度 /度 ======== -->
     <xacro:property name="rad_30" value="${30 * pi / 180.0}"/>

File: src/raphael_robot_description/urdf/10_snake/69_snake_robot.xacro (robot description, xacro)
@@ -1,6 +1,8 @@
 <?xml version="1.0"?>
 <robot name="snake_robot" xmlns:xacro="http://www.ros.org/wiki/xacro">
-    <!-- 10 加载snake材质 -->
-    <xacro:include filename="$(find raphael_robot_description)/urdf/10_snake/01_snake_materials.xacro"/>
+    <!--  00 加载 inertia 宏定义-->
+    <xacro:include filename="00_snake_inertia.xacro"/>
+    <!-- 00 加载snake材质 -->
+    <xacro:include filename="00_snake_materials.xacro"/>
     <!-- 11 stl模型缩1000倍，单位转为 米 -->
     <xacro:property name="mesh_scale" value="0.001 0.001 0.001"/>
@@ -8,9 +10,9 @@
     <xacro:property name="stl_path" value="package://raphael_robot_description/meshes/snake"/>
     <!-- 13 各连杆的质量、外径、长度 -->
-    <xacro:include filename="$(find raphael_robot_description)/urdf/10_snake/00_snake_params.xacro"/>
+    <xacro:include filename="00_snake_params.xacro"/>
     <!-- 14 创建连杆的函数 -->
-    <xacro:include filename="$(find raphael_robot_description)/urdf/10_snake/10_snake_links.xacro"/>
+    <xacro:include filename="10_snake_links.xacro"/>
     <!-- 15 创建关节的函数 -->
-    <xacro:include filename="$(find raphael_robot_description)/urdf/10_snake/11_snake_joints.xacro"/>
+    <xacro:include filename="11_snake_joints.xacro"/>
     <!-- 16 调用宏生成snake -->
     <xacro:get_snake_links prefix="s1"/>

File: src/raphael_robot_description/urdf/10_snake/99_snake_robot.urdf.xacro (robot description, xacro)
@@ -1,4 +1,4 @@
 <?xml version="1.0"?>
-<robot name="snake_robot" xmlns:xacro="http://www.ros.org/wiki/xacro">
+<robot xmlns:xacro="http://www.ros.org/wiki/xacro">
     <xacro:include filename="69_snake_robot.xacro"/>
     <xacro:include filename="89_snake_robot.ros2_control.xacro"/>

File: src/raphael_robot_description/urdf/40_tricycle/00_tricycle_inertia.xacro (robot description, xacro)
@@ -2,5 +2,5 @@
 <robot xmlns:xacro="http://www.ros.org/wiki/xacro">
     <!-- 长方体惯性宏           params: m质量(kg), x/y/z长宽高(m), o_xyz重心偏移, o_rpy重心姿态 -->
-    <xacro:macro name="box_inertia" params="m x y z o_xyz o_rpy">
+    <xacro:macro name="tricycle_box_inertia" params="m x y z o_xyz o_rpy">
         <inertial>
             <mass value="${m}"/>
@@ -12,5 +12,5 @@
     </xacro:macro>
     <!-- 实心圆柱惯性宏（杆轴线沿Z）params: m质量(kg), r外半径(m), l杆长(m), o_xyz重心偏移, o_rpy重心姿态   -->
-    <xacro:macro name="cylinder_inertia" params="m r l o_xyz o_rpy">
+    <xacro:macro name="tricycle_cylinder_inertia" params="m r l o_xyz o_rpy">
         <inertial>
             <mass value="${m}"/>
@@ -22,5 +22,5 @@
     </xacro:macro>
     <!-- 实心球体惯性宏  params: m质量(kg), r球半径(m), o_xyz重心偏移, o_rpy重心姿态  -->
-    <xacro:macro name="sphere_inertia" params="m r o_xyz o_rpy">
+    <xacro:macro name="tricycle_sphere_inertia" params="m r o_xyz o_rpy">
         <inertial>
             <mass value="${m}"/>
@@ -32,5 +32,5 @@
     </xacro:macro>
     <!-- 空心圆筒惯性宏（轴线沿Z） params: m总质量(kg), r_out外半径(m), r_in内孔半径(m), l杆长(m), o_xyz重心偏移, o_rpy重心姿态 -->
-    <xacro:macro name="hollow_cylinder_inertia" params="m r_out r_in l o_xyz o_rpy">
+    <xacro:macro name="tricycle_hollow_cylinder_inertia" params="m r_out r_in l o_xyz o_rpy">
         <inertial>
             <mass value="${m}"/>

File: src/raphael_robot_description/urdf/40_tricycle/69_mobile_base.xacro (robot description, xacro)
@@ -7,7 +7,9 @@
     <xacro:property name="wheel_radius" value="0.1"/>
     <xacro:property name="wheel_length" value="0.05"/>
-    <!-- 🎯 全局缩放系数（修改此值即可整体缩放） -->
+    <!-- 🎯 全局缩放系数 -->
     <xacro:property name="scale" value="0.1"/>
+    <!-- ========== 基座 footprint ========== -->
     <link name="base_footprint_tricycle"/>
+    <!-- ========== base_link ========== -->
     <link name="base_link">
         <visual>
@@ -18,7 +20,17 @@
             <material name="blue"/>
         </visual>
+        <collision>
+            <geometry>
+                <box size="${base_length * scale} ${base_width * scale} ${base_height * scale}"/>
+            </geometry>
+            <origin xyz="0 0 ${base_height * scale / 2.0}" rpy="0 0 0"/>
+        </collision>
+        <xacro:tricycle_box_inertia m="200.0" x="${base_length*scale}" y="${base_width*scale}" z="${base_height*scale}"
+                                    o_xyz="0 0 ${base_height*scale/2.0}" o_rpy="0 0 0"/>
     </link>
+    <!-- ========== 轮子宏 ========== -->
     <xacro:macro name="wheel_link" params="prefix">
         <link name="${prefix}_wheel_link">
+            <!-- 视觉：圆柱 -->
             <visual>
                 <geometry>
@@ -28,8 +40,18 @@
                 <material name="grey"/>
             </visual>
+            <!-- 碰撞：球体 -->
+            <collision>
+                <geometry>
+                    <sphere radius="${wheel_radius * scale}"/>
+                </geometry>
+                <origin xyz="0 0 0" rpy="0 0 0"/>
+            </collision>
+            <xacro:tricycle_cylinder_inertia m="10" r="${wheel_radius*scale}" l="${wheel_length*scale}" o_xyz="0 0 0" o_rpy="0 0 0"/>
         </link>
     </xacro:macro>
+    <!-- 实例化左右轮子 -->
     <xacro:wheel_link prefix="right"/>
     <xacro:wheel_link prefix="left"/>
+    <!-- ========== 万向轮（脚轮） ========== -->
     <link name="caster_wheel_link">
         <visual>
@@ -40,5 +62,13 @@
             <material name="grey"/>
         </visual>
+        <collision>
+            <geometry>
+                <sphere radius="${wheel_radius * scale / 2.0}"/>
+            </geometry>
+            <origin xyz="0 0 0" rpy="0 0 0"/>
+        </collision>
+        <xacro:tricycle_sphere_inertia m="10" r="${wheel_radius*scale/2.0}" o_xyz="0 0 0" o_rpy="0 0 0"/>
     </link>
+    <!-- ========== 关节 ========== -->
     <joint name="base_tricycle_joint" type="fixed">
         <parent link="base_footprint_tricycle"/>

File: src/raphael_robot_description/urdf/40_tricycle/99_tricycle_robot.urdf.xacro (robot description, xacro)
@@ -1,6 +1,7 @@
 <?xml version="1.0"?>
-<robot name="my_robot" xmlns:xacro="http://www.ros.org/wiki/xacro">
+<robot xmlns:xacro="http://www.ros.org/wiki/xacro">
     <xacro:include filename="00_common_properties.xacro"/>
+    <xacro:include filename="00_tricycle_inertia.xacro"/>
     <xacro:include filename="69_mobile_base.xacro"/>
-    <xacro:include filename="89_mobile_base.ros2_control.xacro"/>
+    <xacro:include filename="89_tricycle_gazebo.xacro"/>
 </robot>

File: src/raphael_robot_description/urdf/raphael_robot.urdf.xacro (robot description, xacro)
@@ -17,3 +17,7 @@
         <origin xyz="0 0 0.033" rpy="0 0 0"/>
     </joint>
+    <gazebo>
+        <plugin filename="gz_ros2_control-system" name="gz_ros2_control::GazeboSimROS2ControlPlugin">
+        <parameters>$(find raphael_robot)/config/tricycle_control.yaml</parameters>
+    </gazebo>
 </robot>
