Commit message: 小车模拟驱动，snake的5个关节电机由电机驱动。 forward_command_controller/ForwardCommandController这个控制器初始角度是NAN

File: src/raphael_robot_description/urdf/10_snake/89_snake_robot.ros2_control.xacro (robot description, xacro)
@@ -1,36 +1,36 @@
 <?xml version="1.0"?>
 <robot xmlns:xacro="http://www.ros.org/wiki/xacro">
-    <!--    <ros2_control name="SnakeHardware" type="system">-->
-    <!--        <hardware>-->
-    <!--            <plugin>snake_hardware/SnakeHardwareInterface</plugin>-->
-    <!--            <param name="st3215_port">/dev/ttyACM0</param>-->
-    <!--            <param name="baud">1000000</param>-->
-    <!--            <param name="s1_motor_06_07">6</param>-->
-    <!--            <param name="s1_motor_07_08">7</param>-->
-    <!--            <param name="s1_motor_08_09">8</param>-->
-    <!--            <param name="s1_motor_09b_10">9</param>-->
-    <!--            <param name="s1_motor_10_11">10</param>-->
-    <!--        </hardware>-->
-    <!--        <joint name="s1_link06_link07_joint">-->
-    <!--            <command_interface name="position"/>-->
-    <!--            <state_interface name="position"/>-->
-    <!--        </joint>-->
-    <!--        <joint name="s1_link07_link08_joint">-->
-    <!--            <command_interface name="position"/>-->
-    <!--            <state_interface name="position"/>-->
-    <!--        </joint>-->
-    <!--        <joint name="s1_link08_link09_joint">-->
-    <!--            <command_interface name="position"/>-->
-    <!--            <state_interface name="position"/>-->
-    <!--        </joint>-->
-    <!--        <joint name="s1_link09b_link10_joint">-->
-    <!--            <command_interface name="position"/>-->
-    <!--            <state_interface name="position"/>-->
-    <!--        </joint>-->
-    <!--        <joint name="s1_link10_link11_joint">-->
-    <!--            <command_interface name="position"/>-->
-    <!--            <state_interface name="position"/>-->
-    <!--        </joint>-->
-    <!--    </ros2_control>-->
+    <ros2_control name="SnakeHardware" type="system">
+        <hardware>
+            <plugin>snake_hardware/SnakeHardwareInterface</plugin>
+            <param name="st3215_port">/dev/ttyACM0</param>
+            <param name="baud">1000000</param>
+            <param name="s1_motor_06_07">6</param>
+            <param name="s1_motor_07_08">7</param>
+            <param name="s1_motor_08_09">8</param>
+            <param name="s1_motor_09b_10">9</param>
+            <param name="s1_motor_10_11">10</param>
+        </hardware>
+        <joint name="s1_link06_link07_joint">
+            <command_interface name="position"/>
+            <state_interface name="position"/>
+        </joint>
+        <joint name="s1_link07_link08_joint">
+            <command_interface name="position"/>
+            <state_interface name="position"/>
+        </joint>
+        <joint name="s1_link08_link09_joint">
+            <command_interface name="position"/>
+            <state_interface name="position"/>
+        </joint>
+        <joint name="s1_link09b_link10_joint">
+            <command_interface name="position"/>
+            <state_interface name="position"/>
+        </joint>
+        <joint name="s1_link10_link11_joint">
+            <command_interface name="position"/>
+            <state_interface name="position"/>
+        </joint>
+    </ros2_control>
     <!--    仿真/Mock 硬件接口配置-->
     <ros2_control name="SnakeHardwareMock" type="system">
@@ -64,24 +64,24 @@
         </joint>
         <!--  ========================== 以下就有足够的电机可以匹配了 ========================-->
-        <joint name="s1_link06_link07_joint">-->
-            <command_interface name="position"/>
-            <state_interface name="position"/>
-        </joint>
-        <joint name="s1_link07_link08_joint">
-            <command_interface name="position"/>
-            <state_interface name="position"/>
-        </joint>
-        <joint name="s1_link08_link09_joint">
-            <command_interface name="position"/>
-            <state_interface name="position"/>
-        </joint>
-        <joint name="s1_link09b_link10_joint">
-            <command_interface name="position"/>
-            <state_interface name="position"/>
-        </joint>
-        <joint name="s1_link10_link11_joint">
-            <command_interface name="position"/>
-            <state_interface name="position"/>
-        </joint>
+        <!--        <joint name="s1_link06_link07_joint">&ndash;&gt;-->
+        <!--            <command_interface name="position"/>-->
+        <!--            <state_interface name="position"/>-->
+        <!--        </joint>-->
+        <!--        <joint name="s1_link07_link08_joint">-->
+        <!--            <command_interface name="position"/>-->
+        <!--            <state_interface name="position"/>-->
+        <!--        </joint>-->
+        <!--        <joint name="s1_link08_link09_joint">-->
+        <!--            <command_interface name="position"/>-->
+        <!--            <state_interface name="position"/>-->
+        <!--        </joint>-->
+        <!--        <joint name="s1_link09b_link10_joint">-->
+        <!--            <command_interface name="position"/>-->
+        <!--            <state_interface name="position"/>-->
+        <!--        </joint>-->
+        <!--        <joint name="s1_link10_link11_joint">-->
+        <!--            <command_interface name="position"/>-->
+        <!--            <state_interface name="position"/>-->
+        <!--        </joint>-->
     </ros2_control>
 </robot>

File: src/raphael_robot_description/urdf/40_tricycle/89_mobile_base.ros2_control.xacro (robot description, xacro)
@@ -2,15 +2,15 @@
 <robot xmlns:xacro="http://www.ros.org/wiki/xacro">
     <ros2_control name="TricycleHardware" type="system">
+        <hardware>
+            <plugin>mock_components/GenericSystem</plugin>
+            <param name="calculate_dynamics">true</param>
+        </hardware>
         <!--        <hardware>-->
-        <!--            <plugin>mock_components/GenericSystem</plugin>-->
-        <!--            <param name="calculate_dynamics">true</param>-->
+        <!--            <plugin>tricycle_hardware/TricycleHardwareInterface</plugin>-->
+        <!--            <param name="left_motor_id">9</param>-->
+        <!--            <param name="right_motor_id">10</param>-->
+        <!--            <param name="baud">1000000</param>-->
+        <!--            <param name="st3215_port">/dev/ttyACM0</param>-->
         <!--        </hardware>-->
-        <hardware>
-            <plugin>tricycle_hardware/TricycleHardwareInterface</plugin>
-            <param name="left_motor_id">9</param>
-            <param name="right_motor_id">10</param>
-            <param name="baud">1000000</param>
-            <param name="st3215_port">/dev/ttyACM0</param>
-        </hardware>
         <joint name="base_right_wheel_joint">
             <command_interface name="velocity"/>

Commit message: udemy上的ros2_control学习完毕

File: src/raphael_robot_description/urdf/10_snake/89_snake_robot.ros2_control.xacro (robot description, xacro)
@@ -2,4 +2,8 @@
 <robot xmlns:xacro="http://www.ros.org/wiki/xacro">
     <ros2_control name="SnakeHardware" type="system">
+        <!--        <hardware>-->
+        <!--            <plugin>mock_components/GenericSystem</plugin>-->
+        <!--            <param name="calculate_dynamics">true</param>-->
+        <!--        </hardware>-->
         <hardware>
             <plugin>snake_hardware/SnakeHardwareInterface</plugin>
@@ -63,25 +67,4 @@
             <state_interface name="position"/>
         </joint>
-        <!--  ========================== 以下就有足够的电机可以匹配了 ========================-->
-        <!--        <joint name="s1_link06_link07_joint">&ndash;&gt;-->
-        <!--            <command_interface name="position"/>-->
-        <!--            <state_interface name="position"/>-->
-        <!--        </joint>-->
-        <!--        <joint name="s1_link07_link08_joint">-->
-        <!--            <command_interface name="position"/>-->
-        <!--            <state_interface name="position"/>-->
-        <!--        </joint>-->
-        <!--        <joint name="s1_link08_link09_joint">-->
-        <!--            <command_interface name="position"/>-->
-        <!--            <state_interface name="position"/>-->
-        <!--        </joint>-->
-        <!--        <joint name="s1_link09b_link10_joint">-->
-        <!--            <command_interface name="position"/>-->
-        <!--            <state_interface name="position"/>-->
-        <!--        </joint>-->
-        <!--        <joint name="s1_link10_link11_joint">-->
-        <!--            <command_interface name="position"/>-->
-        <!--            <state_interface name="position"/>-->
-        <!--        </joint>-->
     </ros2_control>
 </robot>

File: src/raphael_robot_description/urdf/40_tricycle/99_tricycle_robot.urdf.xacro (robot description, xacro)
@@ -4,4 +4,4 @@
     <xacro:include filename="00_tricycle_inertia.xacro"/>
     <xacro:include filename="69_mobile_base.xacro"/>
-    <xacro:include filename="89_tricycle_gazebo.xacro"/>
+    <xacro:include filename="89_mobile_base.ros2_control.xacro"/>
 </robot>

File: src/raphael_robot_description/urdf/raphael_robot.urdf.xacro (robot description, xacro)
@@ -17,7 +17,3 @@
         <origin xyz="0 0 0.033" rpy="0 0 0"/>
     </joint>
-    <gazebo>
-        <plugin filename="gz_ros2_control-system" name="gz_ros2_control::GazeboSimROS2ControlPlugin">
-        <parameters>$(find raphael_robot)/config/tricycle_control.yaml</parameters>
-    </gazebo>
 </robot>
