Commit message: fd_left_hardware包已创建

File: src/raphael_robot/fd_left_robot/fd_left_description/config/fd.config.xacro (robot description, xacro)
@@ -2,28 +2,28 @@
 <robot xmlns:xacro="http://www.ros.org/wiki/xacro" name="fd">
     <!-- Parameters -->
-    <xacro:arg name="robot_id" default="fd"/> <!-- Name of the haptic interface -->
+    <xacro:arg name="robot_id" default="fd_left"/> <!-- Name of the haptic interface -->
     <xacro:arg name="use_fake_hardware" default="false"/>
-    <xacro:arg name="use_orientation" default="false"/>
-    <xacro:arg name="use_clutch" default="false"/>
+    <xacro:arg name="use_orientation" default="true"/>
+    <xacro:arg name="use_clutch" default="true"/>
     <!-- Import interface urdf file -->
-    <xacro:include filename="$(find fd_description)/urdf/fd.urdf.xacro"/>
+    <xacro:include filename="$(find fd_left_description)/urdf/fd.urdf.xacro"/>
     <xacro:haptic_interface
-    	robot_id="$(arg robot_id)"
-    	use_orientation="$(arg use_orientation)"
-    	use_clutch="$(arg use_clutch)"
+            robot_id="$(arg robot_id)"
+            use_orientation="$(arg use_orientation)"
+            use_clutch="$(arg use_clutch)"
     />
     <!-- Import and setup interface ros2_control description -->
-    <xacro:include filename="$(find fd_description)/ros2_control/fd.r2c_hardware.xacro" />
+    <xacro:include filename="$(find fd_left_description)/ros2_control/fd.r2c_hardware.xacro"/>
     <xacro:fd_ros2_control
-        interface_id="-1"
-        interface_sn="-1"
-        robot_id= "$(arg robot_id)"
-        use_fake_hardware="$(arg use_fake_hardware)"
-        use_orientation="$(arg use_orientation)"
-    	orientation_is_actuated="$(arg use_orientation)"
-        ignore_orientation_readings="false"
-        use_clutch="$(arg use_clutch)"
-        emulate_button="true"
-        effector_mass="-1.0"
+            interface_id="-1"
+            interface_sn="-1"
+            robot_id="$(arg robot_id)"
+            use_fake_hardware="$(arg use_fake_hardware)"
+            use_orientation="$(arg use_orientation)"
+            orientation_is_actuated="$(arg use_orientation)"
+            ignore_orientation_readings="false"
+            use_clutch="$(arg use_clutch)"
+            emulate_button="true"
+            effector_mass="-1.0"
     />
     <!-- Default effector masses:

File: src/raphael_robot/fd_left_robot/fd_left_description/urdf/fd.urdf.xacro (robot description, xacro)
@@ -16,5 +16,5 @@
             <child link="${robot_id}_x_link"/>
             <axis xyz="1 0 0"/>
-            <limit effort="12" velocity="1.0" lower="-2" upper="2" />
+            <limit effort="12" velocity="1.0" lower="-2" upper="2"/>
         </joint>
         <joint name="${robot_id}_y" type="prismatic">
@@ -23,5 +23,5 @@
             <child link="${robot_id}_y_link"/>
             <axis xyz="0 1 0"/>
-            <limit effort="12" velocity="1.0" lower="-2" upper="2" />
+            <limit effort="12" velocity="1.0" lower="-2" upper="2"/>
         </joint>
         <joint name="${robot_id}_z" type="prismatic">
@@ -30,13 +30,14 @@
             <child link="${robot_id}_z_link"/>
             <axis xyz="0 0 1"/>
-            <limit effort="12" velocity="1.0" lower="-2" upper="2" />
+            <limit effort="12" velocity="1.0" lower="-2" upper="2"/>
         </joint>
         <!-- Orientation from XYZ roll-pitch-yaw angles -->
         <!-- TODO: change when/if floating joints are supported by ros2 control AND KDL -->
+        <!--  是不是要三个方向的旋转？ 如果要，value = revolute, 否则 value = fixed-->
         <xacro:if value="${use_orientation}">
-            <xacro:property name="orientation_joint_type" value="revolute" />
+            <xacro:property name="orientation_joint_type" value="revolute"/>
         </xacro:if>
         <xacro:unless value="${use_orientation}">
-            <xacro:property name="orientation_joint_type" value="fixed" />
+            <xacro:property name="orientation_joint_type" value="fixed"/>
         </xacro:unless>
         <joint name="${robot_id}_roll" type="${orientation_joint_type}">
@@ -45,5 +46,5 @@
             <child link="${robot_id}_roll_link"/>
             <axis xyz="1 0 0"/>
-            <limit effort="0.4" velocity="10.0" lower="-${pi}" upper="${pi}" />
+            <limit effort="0.4" velocity="10.0" lower="-${pi}" upper="${pi}"/>
         </joint>
         <joint name="${robot_id}_pitch" type="${orientation_joint_type}">
@@ -52,5 +53,5 @@
             <child link="${robot_id}_pitch_link"/>
             <axis xyz="0 1 0"/>
-            <limit effort="0.4" velocity="10.0" lower="-${pi}" upper="${pi}" />
+            <limit effort="0.4" velocity="10.0" lower="-${pi}" upper="${pi}"/>
         </joint>
         <joint name="${robot_id}_yaw" type="${orientation_joint_type}">
@@ -59,5 +60,5 @@
             <child link="${robot_id}_yaw_link"/>
             <axis xyz="0 0 1"/>
-            <limit effort="0.4" velocity="10.0" lower="-${pi}" upper="${pi}" />
+            <limit effort="0.4" velocity="10.0" lower="-${pi}" upper="${pi}"/>
         </joint>
         <!-- Tool -->
@@ -75,6 +76,6 @@
                 <child link="${robot_id}_virtual_clutch_link"/>
                 <axis xyz="1 0 0"/>
-            <limit effort="12" velocity="1.0" lower="-0.05" upper="0.05" />
-        </joint>
+                <limit effort="12" velocity="1.0" lower="-0.05" upper="0.05"/>
+            </joint>
         </xacro:if>
     </xacro:macro>
