Commit message: 完成fd_left的hardware

File: src/raphael_description/urdf/MTM/fd_left/fd_left.config.xacro (robot description, xacro)
@@ -5,5 +5,5 @@
     <xacro:arg name="use_fake_hardware" default="false"/>
     <xacro:arg name="use_orientation" default="true"/>
-    <xacro:arg name="use_clutch" default="true"/>
+    <xacro:arg name="use_gripper" default="true"/>
     <!-- Import interface urdf file -->
     <xacro:include filename="$(find raphael_description)/urdf/MTM/fd_left/fd_left.urdf.xacro"/>
@@ -11,5 +11,5 @@
             robot_id="$(arg robot_id)"
             use_orientation="$(arg use_orientation)"
-            use_clutch="$(arg use_clutch)"
+            use_gripper="$(arg use_gripper)"
     />
     <!-- Import and setup interface ros2_control description -->
@@ -23,5 +23,5 @@
             orientation_is_actuated="$(arg use_orientation)"
             ignore_orientation_readings="false"
-            use_clutch="$(arg use_clutch)"
+            use_gripper="$(arg use_gripper)"
             emulate_button="true"
             effector_mass="-1.0"

File: src/raphael_description/urdf/MTM/fd_left/fd_left.r2c_hardware.xacro (robot description, xacro)
@@ -2,6 +2,6 @@
 <robot xmlns:xacro="http://www.ros.org/wiki/xacro">
     <xacro:macro
-        name="fd_ros2_control"
-        params="robot_id plugin_name:='FDHapticInterface' interface_id:='-1' interface_sn:='-1' effector_mass:='-1.0' use_fake_hardware:='false' use_orientation:='false' orientation_is_actuated:='false' use_clutch:='false' emulate_button:='false' ignore_orientation_readings:='false'">
+            name="fd_ros2_control"
+            params="robot_id plugin_name:='FDHapticInterface' interface_id:='-1' interface_sn:='-1' effector_mass:='-1.0' use_fake_hardware:='false' use_orientation:='false' orientation_is_actuated:='false' use_gripper:='false' emulate_button:='false' ignore_orientation_readings:='false'">
         <ros2_control name="${plugin_name}" type="system">
             <hardware>
@@ -51,7 +51,7 @@
                 <xacro:configure_rotation_joint joint_name="${robot_id}_yaw"/>
             </xacro:if>
-            <!-- Configure clutch -->
-            <xacro:if value="${use_clutch}">
-                <xacro:configure_translation_joint joint_name="${robot_id}_clutch"/>
+            <!-- Configure gripper -->
+            <xacro:if value="${use_gripper}">
+                <xacro:configure_translation_joint joint_name="${robot_id}_gripper"/>
             </xacro:if>
         </ros2_control>

File: src/raphael_description/urdf/MTM/fd_left/fd_left.urdf.xacro (robot description, xacro)
@@ -1,5 +1,5 @@
 <?xml version="1.0" encoding='utf-8'?>
 <robot xmlns:xacro="http://www.ros.org/wiki/xacro" name="fd">
-    <xacro:macro name="haptic_interface" params="robot_id:='fd' use_orientation:='false' use_clutch:='false'">
+    <xacro:macro name="haptic_interface" params="robot_id:='fd' use_orientation:='false' use_gripper:='false'">
         <link name="${robot_id}_base"/>
         <link name="${robot_id}_x_link"/>
@@ -16,5 +16,5 @@
             <child link="${robot_id}_x_link"/>
             <axis xyz="1 0 0"/>
-            <limit effort="12" velocity="1.0" lower="-2" upper="2" />
+            <limit effort="12" velocity="1.0" lower="-2" upper="2"/>
         </joint>
         <joint name="${robot_id}_y" type="prismatic">
@@ -23,5 +23,5 @@
             <child link="${robot_id}_y_link"/>
             <axis xyz="0 1 0"/>
-            <limit effort="12" velocity="1.0" lower="-2" upper="2" />
+            <limit effort="12" velocity="1.0" lower="-2" upper="2"/>
         </joint>
         <joint name="${robot_id}_z" type="prismatic">
@@ -30,13 +30,13 @@
             <child link="${robot_id}_z_link"/>
             <axis xyz="0 0 1"/>
-            <limit effort="12" velocity="1.0" lower="-2" upper="2" />
+            <limit effort="12" velocity="1.0" lower="-2" upper="2"/>
         </joint>
         <!-- Orientation from XYZ roll-pitch-yaw angles -->
         <!-- TODO: change when/if floating joints are supported by ros2 control AND KDL -->
         <xacro:if value="${use_orientation}">
-            <xacro:property name="orientation_joint_type" value="revolute" />
+            <xacro:property name="orientation_joint_type" value="revolute"/>
         </xacro:if>
         <xacro:unless value="${use_orientation}">
-            <xacro:property name="orientation_joint_type" value="fixed" />
+            <xacro:property name="orientation_joint_type" value="fixed"/>
         </xacro:unless>
         <joint name="${robot_id}_roll" type="${orientation_joint_type}">
@@ -45,5 +45,5 @@
             <child link="${robot_id}_roll_link"/>
             <axis xyz="1 0 0"/>
-            <limit effort="0.4" velocity="10.0" lower="-${pi}" upper="${pi}" />
+            <limit effort="0.4" velocity="10.0" lower="-${pi}" upper="${pi}"/>
         </joint>
         <joint name="${robot_id}_pitch" type="${orientation_joint_type}">
@@ -52,5 +52,5 @@
             <child link="${robot_id}_pitch_link"/>
             <axis xyz="0 1 0"/>
-            <limit effort="0.4" velocity="10.0" lower="-${pi}" upper="${pi}" />
+            <limit effort="0.4" velocity="10.0" lower="-${pi}" upper="${pi}"/>
         </joint>
         <joint name="${robot_id}_yaw" type="${orientation_joint_type}">
@@ -59,5 +59,5 @@
             <child link="${robot_id}_yaw_link"/>
             <axis xyz="0 0 1"/>
-            <limit effort="0.4" velocity="10.0" lower="-${pi}" upper="${pi}" />
+            <limit effort="0.4" velocity="10.0" lower="-${pi}" upper="${pi}"/>
         </joint>
         <!-- Tool -->
@@ -67,14 +67,14 @@
             <child link="${robot_id}_ee"/>
         </joint>
-        <!-- Clutch -->
-        <xacro:if value="${use_clutch}">
-            <link name="${robot_id}_virtual_clutch_link"/>
-            <joint name="${robot_id}_clutch" type="prismatic">
+        <!-- gripper -->
+        <xacro:if value="${use_gripper}">
+            <link name="${robot_id}_virtual_gripper_link"/>
+            <joint name="${robot_id}_gripper" type="prismatic">
                 <origin rpy="0 0 0" xyz="0 0 0"/>
                 <parent link="${robot_id}_ee"/>
-                <child link="${robot_id}_virtual_clutch_link"/>
+                <child link="${robot_id}_virtual_gripper_link"/>
                 <axis xyz="1 0 0"/>
-            <limit effort="12" velocity="1.0" lower="-0.05" upper="0.05" />
-        </joint>
+                <limit effort="12" velocity="1.0" lower="-0.05" upper="0.05"/>
+            </joint>
         </xacro:if>
     </xacro:macro>
